Commit message: 3rd update

File: clearpath_common/clearpath_platform_description/urdf/a200/attachments/top_plate.urdf.xacro (robot description, xacro)
@@ -112,5 +112,5 @@
         <link name="ur_base_link">
           <visual>
-            <origin xyz="-0.3 0 -0.07" rpy="0 0 0" />
+            <origin xyz="-0.2 0 -0.07" rpy="0 0 0" />
             <geometry>
               <mesh filename="package://clearpath_platform_description/meshes/a200/attachments/husky_frame_vi.stl" />
@@ -119,5 +119,5 @@
           </visual>
           <collision>
-            <origin xyz="-0.3 0 -0.07" rpy="0 0 0"/>
+            <origin xyz="-0.2 0 -0.07" rpy="0 0 0"/>
             <geometry>
               <mesh filename="package://clearpath_platform_description/meshes/a200/attachments/husky_frame_co.stl" />
@@ -128,5 +128,5 @@
           <parent link="${name}_default_mount" />
           <child link="ur_base_link"/>
-          <origin xyz="0.3 0 0.07" rpy="0 0 0"/>
+          <origin xyz="0.2 0 0.07" rpy="0 0 0"/>
         </joint>
       </xacro:if>
